File: hardware/rp2040-logic-analyzer.kicad_sch (KiCad schematic)
At the start: 79 parts, among them J1 TYPE-C-31-M-12, J2 PROBE 2x16, J3 VREF_EXT, J4 ADC 1x3 (DNF), SW1 SK13D07VG5, SW2 TS-1187A-B-A-B, SW3 TS-1187A-B-A-B, U1 RP2040, U2 W25Q128JVSIQ, U3 TXU0104PWR, U4 TXU0104PWR, U5 TXU0104PWR, U6 TXU0104PWR, U7 AMS1117-3.3, U8 USBLC6-2SC6, X1 ABM8-272-T3 12MHz

Commit message: PCB 第1版: 配置済み・未配線の基板と生成/配線/出力ツール（回路図に TP8/TP9・C27 追加）
- tools/gen_pcb.py: ネットリストから .kicad_pcb を生成（4層 JLC04161H-7628・KIT §3 の DRC/ネットクラス・配置表・USB 差動手配線・内層 GND/+3V3 plane）
- tools/route_pcb.py: freerouting 駆動（--input で人間の版・--pours-only で配線後に B.Cu GND ベタ）
- tools/make_outputs.py: DRC → Gerber/Drill/CPL/zip/render（未実行・人間の配線後）
- hardware/: 配置済み基板（DRC error 0・未配線 192＝配線前）。out/placed・out/route（freerouting 試行の参考）
- 回路図: TP8=SWCLK・TP9=SWDIO・C27 1µF(VREF) を追加（ERC 0・照合 88・KIT 17 項目 PASS）

Co-Authored-By: Claude Opus 5 (1M context) <noreply@anthropic.com>
Claude-Session: https://claude.ai/code/session_01QcyfLK5Dm75FgDGZMr6fff
Parts:
- added C27: 1µF, Capacitor_SMD:C_0402_1005Metric, symbol Device:C
- added TP8: SWCLK, TestPoint:TestPoint_Pad_1.0x1.0mm, symbol Connector:TestPoint
- added TP9: SWDIO, TestPoint:TestPoint_Pad_1.0x1.0mm, symbol Connector:TestPoint
Connections:
- net GND: now also C27.2
- net VREF: now also C27.1
- net SWCLK: now reaches U1.24 (SWCLK)
- net SWCLK: now also TP8.1
- net SWDIO: now reaches U1.25 (SWDIO)
- net SWDIO: now also TP9.1
- no-connect marks 16 -> 14
Other:
- note added: "DNF: R23 (10k QSPI_SS pull-up), J4 (analog header). SWD on test pads TP8 (SWCLK) / TP9 (SWDIO). C27 = 1uF bulk on VREF."
- note added: "U1 RP2040 + U2 W25Q128 (QSPI) + X1 12MHz ; 100nF x10 (C1-C10) + 1uF x2 (C21/C22) ; BOOT = SW2, RUN = SW3 ; SWD on TP8/TP9"
- note removed: "DNF: R23 (10k QSPI_SS pull-up), J4 (analog header). SWCLK/SWDIO not brought out (KIT §5-15, open item)."
- note removed: "U1 RP2040 + U2 W25Q128 (QSPI) + X1 12MHz ; 100nF x10 (C1-C10) + 1uF x2 (C21/C22) ; BOOT = SW2, RUN = SW3"

Commit message: 人間の GUI 編集を取り込み（PCB: 微細ピッチのファンアウト配線 10 本＋ビア 5・回路図の整形）
Co-Authored-By: Claude Opus 5 (1M context) <noreply@anthropic.com>
Claude-Session: https://claude.ai/code/session_01QcyfLK5Dm75FgDGZMr6fff
Other:
- moved on the sheet: J4
