File: hardware/rp2040-logic-analyzer.kicad_sch (KiCad schematic)
At the start: 82 parts, among them J1 TYPE-C-31-M-12, J2 PROBE 2x16, J3 VREF_EXT, J4 ADC 1x3 (DNF), SW1 SK13D07VG5, SW2 TS-1187A-B-A-B, SW3 TS-1187A-B-A-B, U1 RP2040, U2 W25Q128JVSIQ, U3 TXU0104PWR, U4 TXU0104PWR, U5 TXU0104PWR, U6 TXU0104PWR, U7 AMS1117-3.3, U8 USBLC6-2SC6, X1 ABM8-272-T3 12MHz

Commit message: SW1（SK13D07VG5）のコモンをピン 2 に訂正: シンボルのピン番号・SPEC §5.4/§17・KICAD-KIT・tools の期待値・図を更新（実測 2026-10-04）
Connections:
- net +3V3: now also SW1.1; no longer SW1.2
- net VREF: now also SW1.2 (COM); no longer SW1.1 (COM)
Other:
- note added: "SW1 (SK13D07VG5) is a SHORTING slide switch: +3V3 (pin 1) and +5V (pin 4) are never adjacent; EXT (pin 3) sits between. Do not slide with EXT connected."
- note removed: "SW1 (SK13D07VG5) is a SHORTING slide switch: +3V3 (pin 2) and +5V (pin 4) are never adjacent; EXT (pin 3) sits between. Do not slide with EXT connected."
Changed lines of the file:
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@@
 		)
 	)
-	(text "SW1 (SK13D07VG5) is a SHORTING slide switch: +3V3 (pin 2) and +5V (pin 4) are never adjacent; EXT (pin 3) sits between. Do not slide with EXT connected."
+	(text "SW1 (SK13D07VG5) is a SHORTING slide switch: +3V3 (pin 1) and +5V (pin 4) are never adjacent; EXT (pin 3) sits between. Do not slide with EXT connected."
 		(exclude_from_sim no)
 		(at 12.7 257.81 0)
