File: hardware/rp2040-logic-analyzer.kicad_pcb (KiCad board)
At the start: 4 copper layers, 65 x 45 mm, 82 parts, among them J1 TYPE-C-31-M-12, J2 PROBE 2x16, J3 VREF_EXT, J4 ADC 1x3 (DNF), SW1 SK13D07VG5, SW2 TS-1187A-B-A-B, SW3 TS-1187A-B-A-B, U1 RP2040, U2 W25Q128JVSIQ, U3 TXU0104PWR, U4 TXU0104PWR, U5 TXU0104PWR, U6 TXU0104PWR, U7 AMS1117-3.3, U8 USBLC6-2SC6, X1 ABM8-272-T3 12MHz

Commit message: A1: fix SW1 net assignment (pad1=+3V3, pad2=VREF) and regenerate manufacturing data
- PCB: SW1 pad1/pad2 nets now match the corrected schematic (COM = pad2);
  VREF trace re-routed to pad2, In2 +3V3 plane refilled; silk "RP2040 LA A1",
  back silk "CERN-OHL-P v2"; title block rev A1
- DRC 0 errors / 0 unconnected (47 silk warnings as A0), ERC 0,
  schematic<->board net check 88/88, KIT check 17/17
- hardware/jlcpcb/ now holds A1 (Gerber 16, BOM 19, CPL 68); A0 order data moved to a0/
- make_outputs.py: explicit --excellon-oval-format route (same drill notation as the
  A0 production files); new tools/verify_pcb_netlist.py
- README/SPEC: A1 is untested (not yet manufactured); A0 verified with the rework

Co-Authored-By: Claude Fable 5.1 <noreply@anthropic.com>
Claude-Session: https://claude.ai/code/session_01QcyfLK5Dm75FgDGZMr6fff
Connections:
- SW1 pad 1: VREF -> +3V3
- SW1 pad 2: +3V3 -> VREF
Routing:
- net VREF: track 84.4 -> 86.0 mm
Other:
- board text added: "CERN-OHL-P v2"
- board text added: "RP2040 LA A1"
- board text removed: "RP2040 LA A0"
Changed lines of the file:
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@@
 	(title_block
 		(title "RP2040 16ch Logic Analyzer")
-		(date "2026-09-20")
-		(rev "A0")
+		(date "2026-10-10")
+		(rev "A1")
 		(company "electwork.net")
 		(comment 1 "Generated by tools/gen_pcb.py. CERN-OHL-P-2.0")
@@
 			(layers "*.Cu" "*.Mask")
 			(remove_unused_layers no)
-			(net "VREF")
+			(net "+3V3")
 		)
 		(pad "2" thru_hole circle
@@
 			(layers "*.Cu" "*.Mask")
 			(remove_unused_layers no)
-			(net "+3V3")
+			(net "VREF")
 		)
 		(pad "3" thru_hole circle
@@
 		(layer "Edge.Cuts")
 	)
-	(gr_text "RP2040 LA A0"
+	(gr_text "RP2040 LA A1"
 		(at 105 124.5 0)
 		(layer "F.SilkS")
@@
 		)
 	)
+	(gr_text "CERN-OHL-P v2"
+		(at 132.5 142 0)
+		(layer "B.SilkS")
+		(effects
+			(font
+				(size 1 1)
+				(thickness 0.15)
+			)
+			(justify mirror)
+		)
+	)
 	(segment
 		(start 121.55 128.65)
@@
 	)
 	(segment
-		(start 108.5492 110.1992)
-		(end 107.35 109)
-		(width 0.5)
-		(layer "F.Cu")
-		(net "VREF")
-	)
-	(segment
 		(start 113.1192 113.0992)
 		(end 110.5 110.48)
@@
 	)
 	(segment
+		(start 107.35 111.3984)
+		(end 107.35 113)
+		(width 0.5)
+		(layer "F.Cu")
+		(net "VREF")
+	)
+	(segment
 		(start 119.81 111.08)
 		(end 117.7908 113.0992)
@@
 		(width 0.5)
 		(layer "F.Cu")
+		(net "VREF")
+	)
+	(segment
+		(start 108.5492 110.1992)
+		(end 107.35 111.3984)
+		(width 0.5)
+		(layer "F.Cu")
